File: diy_robotics_arm_pcb/diy_robotics_arm.kicad_pcb (KiCad board)
At the start: 2 copper layers, 125 x 125 mm, 34 parts, among them J1 Conn_01x04, J2 Conn_01x04, J3 Conn_01x04, J4 Conn_01x04, J5 Conn_01x04, J6 Conn_01x04, J7 VCC_ESP32, J8 Enable, J9 VCC_Servos, SW1 SW_DIP_x04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

Commit message: VCC_Servo lable corrected to VCC_Stepper
Parts:
- J9: value VCC_Servos -> VCC_Stepper
Changed lines of the file:
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@@
       (plot_on_all_layers_selection 0x0000000_00000000)
       (disableapertmacros false)
-      (usegerberextensions false)
+      (usegerberextensions true)
       (usegerberattributes true)
       (usegerberadvancedattributes true)
@@
       (psa4output false)
       (plotreference true)
-      (plotvalue true)
+      (plotvalue false)
       (plotinvisibletext false)
       (sketchpadsonfab false)
@@
       (drillshape 0)
       (scaleselection 1)
-      (outputdirectory "")
+      (outputdirectory "fab/")
     )
   )
@@
         (effects (font (size 1 1) (thickness 0.15)))
     )
-    (fp_text value "VCC_Servos" (at 2.5 6.7295) (layer "F.SilkS")
+    (fp_text value "VCC_Stepper" (at 2.5 6.7295) (layer "F.SilkS")
         (effects (font (size 1.5 1.5) (thickness 0.3) bold))
     )
