File: diy_robotics_arm_pcb/diy_robotics_arm.kicad_sch (KiCad schematic)
At the start: 33 parts, among them J1 Conn_01x04, J2 Conn_01x04, J3 Conn_01x04, J4 Conn_01x04, J5 Conn_01x04, J6 Conn_01x04, J7 VCC_ESP32, J8 Enable, J9 VCC_Servos, SW1 SW_DIP_x04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

Commit message: geber files in zip
Other:
- note removed: "A3_STEP war fälschlicherweise auf RXDO (J3-5) anstatt auf IO5"
- note removed: "Check Hardware Enable hinzu"
Changed lines of the file:
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@@
     (effects (font (size 3 3)) (justify left bottom))
-  )
-  (text "Check Hardware\nEnable hinzu" (at 224.79 22.86 0)
-    (effects (font (size 2.54 2.54)) (justify left bottom))
   )
   (text "Achse1" (at 50.8 53.34 0)
@@
     (effects (font (size 1.27 1.27)) (justify left bottom))
   )
-  (text "A3_STEP war \nfälschlicherweise \nauf RXDO (J3-5) \nanstatt auf IO5"
-    (at 247.65 52.07 0)
-    (effects (font (size 2.54 2.54)) (justify left bottom))
-  )
   (text "red\nblue\ngreen\nblack" (at 30.48 167.64 0)

Commit message: VCC_Servo lable corrected to VCC_Stepper
Parts:
- J9: value VCC_Servos -> VCC_Stepper
Changed lines of the file:
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@@
       (effects (font (size 1.27 1.27)))
     )
-    (property "Value" "VCC_Servos" (at 20.32 186.69 0)
+    (property "Value" "VCC_Stepper" (at 20.32 186.69 0)
       (effects (font (size 1.27 1.27)))
     )
